Commit message: with a barely working slam all on raspberry pi

File: mnwlk3r_description/urdf/mnwlk3r_base.xacro (robot description, xacro)
@@ -27,5 +27,5 @@
     <color rgba="1.0 1.0 1.0 1.0"/>
   </material>
-  <gazebo reference="link_chassis">
+  <gazebo reference="base_footprint">
     <material>Gazebo/Orange</material>
   </gazebo>
@@ -41,5 +41,5 @@
                 izz="${mass*(r*r)/2}" />
     </xacro:macro>
-  <link name="link_chassis">
+  <link name="base_footprint">
     <!-- pose and inertial -->
     <pose>0 0 0.068 0 0 0</pose>
@@ -136,5 +136,5 @@
     <origin xyz="0 -0.164 0" rpy="0 0 0"  /> <!-- X=0  |  Y = half box width + 12m spacer + half wheel width ==> x = -280/2 - 12mm -24/2 = -164mm  -->
     <child link="link_right_wheel" />
-    <parent link="link_chassis"/>
+    <parent link="base_footprint"/>
     <axis  xyz="0 1 0" rpy="0 0 0" />
     <limit effort="10000" velocity="1000"/>
@@ -167,5 +167,5 @@
     <origin xyz="0 0.164 0" rpy="0 0 0"  /> <!-- X=0  |  Y = half box width + 12m spacer + half wheel width ==> x = -280/2 - 12mm -24/2 = -164mm  -->
     <child link="link_left_wheel" />
-    <parent link="link_chassis"/>
+    <parent link="base_footprint"/>
     <axis  xyz="0 1 0" rpy="0 0 0" />
     <limit effort="10000" velocity="1000"/>
@@ -198,5 +198,5 @@
     <origin xyz="0.200 0.000 0.110" rpy="0 0 1.5707" />
     <child link="sensor_laser"/>
-    <parent link="link_chassis"/>
+    <parent link="base_footprint"/>
   </joint>
 </robot>
