Commit message: with first rough simulation in gazebo. it seems mnwlk3r kinda 'bounces'...?

File: mnwlk3r_ros/mnwlk3r_description/urdf/mnwlk3r_base.xacro (robot description, xacro)
@@ -33,5 +33,5 @@
   </gazebo>
   <gazebo reference="link_right_wheel">
-    <material>Gazebo/Blue</material>
+    <material>Gazebo/Green</material>
   </gazebo>
     <xacro:macro name="cylinder_inertia" params="mass r l">
@@ -40,4 +40,13 @@
                 izz="${mass*(r*r)/2}" />
     </xacro:macro>
+   <!-- Macro for the inertia of a box
+      source: https://github.com/ethz-asl/rotors_simulator/blob/master/rotors_description/urdf/multirotor_base.xacro
+      note: I am not so sure this formula does apply to me. TODO check against => https://en.wikipedia.org/wiki/List_of_moments_of_inertia
+   -->
+   <xacro:macro name="box_inertia" params="x y z mass">
+     <inertia ixx="${0.0833333 * mass * (y*y + z*z)}" ixy="0.0" ixz="0.0"
+       iyy="${0.0833333 * mass * (x*x + z*z)}" iyz="0.0"
+       izz="${0.0833333 * mass * (x*x + y*y)}" />
+   </xacro:macro>
   <link name="base_footprint">
     <!-- pose and inertial -->
@@ -46,5 +55,6 @@
       <mass value="5"/>
       <origin xyz="0 0 0.1" rpy="0.0 0 0"  />
-      <inertia ixx="0.0395416666667" ixy="0" ixz="0" iyy="0.106208333333" iyz="0" izz="0.106208333333"/>
+      <!-- <inertia ixx="0.0395416666667" ixy="0" ixz="0" iyy="0.106208333333" iyz="0" izz="0.106208333333"/> -->
+      <xacro:box_inertia mass="5.2" x="0.400" y="0.280" z="0.066" />
     </inertial>
     <collision name="collision_chassis">
@@ -64,5 +74,5 @@
     <collision name="caster_front_left_collision">
       <!-- Z = - main wheel radius + caster wheel radius = -136/2 + 63/2 = -68 + 31.5 = -36.5mm  -->
-      <origin xyz="0.200 0.070 -0.0365"  rpy=" 0 0 0"  />
+      <origin xyz="0.200 0.070 -0.0362"  rpy=" 0 0 0"  />
       <geometry>
         <sphere radius="0.0315"/>
@@ -80,5 +90,5 @@
     </collision>
     <visual name="caster_front_left_visual">
-      <origin xyz="0.200 0.070 -0.0365"  rpy=" 0 0 0"  />
+      <origin xyz="0.200 0.070 -0.0362"  rpy=" 0 0 0"  />
       <geometry>
         <sphere radius="0.0315"/>
@@ -87,5 +97,5 @@
     <!-- caster front right  -->
     <collision name="caster_front_right_collision">
-      <origin xyz="0.200 -0.070 -0.0365"  rpy=" 0 0 0"  />
+      <origin xyz="0.200 -0.070 -0.0362"  rpy=" 0 0 0"  />
       <geometry>
         <sphere radius="0.0315"/>
@@ -103,5 +113,53 @@
     </collision>
     <visual name="caster_front_right_visual">
-      <origin xyz="0.200 -0.070 -0.0365"  rpy=" 0 0 0"  />
+      <origin xyz="0.200 -0.070 -0.0362"  rpy=" 0 0 0"  />
+      <geometry>
+        <sphere radius="0.0315"/>
+      </geometry>
+    </visual>
+    <!-- caster back left  -->
+    <collision name="caster_back_left_collision">
+      <!-- Z = - main wheel radius + caster wheel radius = -136/2 + 63/2 = -68 + 31.5 = -36.5mm  -->
+      <origin xyz="-0.150 0.080 -0.0362"  rpy=" 0 0 0"  />
+      <geometry>
+        <sphere radius="0.0315"/>
+      </geometry>
+      <surface>
+        <friction>
+          <ode>
+            <mu>0</mu>
+            <mu2>0</mu2>
+            <slip1>1.0</slip1>
+            <slip2>1.0</slip2>
+          </ode>
+        </friction>
+      </surface>
+    </collision>
+    <visual name="caster_back_left_visual">
+      <origin xyz="-0.150 0.080 -0.0362"  rpy=" 0 0 0"  />
+      <geometry>
+        <sphere radius="0.0315"/>
+      </geometry>
+    </visual>
+    <!-- caster back right  -->
+    <collision name="caster_back_right_collision">
+      <!-- Z = - main wheel radius + caster wheel radius = -136/2 + 63/2 = -68 + 31.5 = -36.5mm  -->
+      <origin xyz="-0.150 -0.080 -0.0362"  rpy=" 0 0 0"  />
+      <geometry>
+        <sphere radius="0.0315"/>
+      </geometry>
+      <surface>
+        <friction>
+          <ode>
+            <mu>0</mu>
+            <mu2>0</mu2>
+            <slip1>1.0</slip1>
+            <slip2>1.0</slip2>
+          </ode>
+        </friction>
+      </surface>
+    </collision>
+    <visual name="caster_back_right_visual">
+      <origin xyz="-0.150 -0.080 -0.0362"  rpy=" 0 0 0"  />
       <geometry>
         <sphere radius="0.0315"/>
@@ -115,5 +173,6 @@
       <mass value="0.2"/>
       <origin  xyz="0 0 0" rpy="1.5707 0 0" />  <!-- only 90 deg rotation on X = pi/2 -->
-      <inertia ixx="0.00052666666" ixy="0" ixz="0" iyy="0.00052666666" iyz="0" izz="0.001"/>
+      <!-- <inertia ixx="0.00052666666" ixy="0" ixz="0" iyy="0.00052666666" iyz="0" izz="0.001"/> -->
+      <xacro:cylinder_inertia mass="0.150" r="${0.136/2}" l="0.024" />
     </inertial>
     <collision name="link_right_wheel_collision">
@@ -146,5 +205,5 @@
       <mass value="0.2"/>
       <origin  xyz="0 0 0" rpy="1.5707 0 0" />  <!-- only 90 deg rotation on X = pi/2 -->
-      <inertia ixx="0.00052666666" ixy="0" ixz="0" iyy="0.00052666666" iyz="0" izz="0.001"/>
+      <xacro:cylinder_inertia mass="0.150" r="${0.136/2}" l="0.024" />
     </inertial>
     <collision name="link_left_wheel_collision">
@@ -195,7 +254,55 @@
   </link>
   <joint name="joint_sensor_laser" type="fixed">
-    <origin xyz="0.200 0.000 0.110" rpy="0 0 1.5707" />
+    <origin xyz="0.200 0.000 0.160" rpy="0 0 1.5707" />
     <child link="sensor_laser"/>
     <parent link="base_footprint"/>
   </joint>
+   <!-- GAZEBO SIMULATION PARAMS / PLUGIN -->
+   <gazebo>
+       <plugin filename="libgazebo_ros_diff_drive.so" name="differential_drive_controller">
+         <alwaysOn>true</alwaysOn>
+         <updateRate>20</updateRate>
+         <leftJoint>joint_left_wheel</leftJoint>
+         <rightJoint>joint_right_wheel</rightJoint>
+         <wheelSeparation>${0.164*2}</wheelSeparation>
+         <wheelDiameter>0.136</wheelDiameter>
+         <torque>0.1</torque>
+         <commandTopic>cmd_vel</commandTopic>
+         <odometryTopic>odom</odometryTopic>
+         <odometryFrame>odom</odometryFrame>
+         <robotBaseFrame>base_footprint</robotBaseFrame>
+         <legacyMode>false</legacyMode>
+       </plugin>
+     </gazebo>
+    <gazebo reference="sensor_laser">  <!-- http://www.theconstructsim.com/ros-projects-exploring-ros-using-2-wheeled-robot-part-1/#part3 -->
+        <sensor type="ray" name="head_rplidar_sensor">
+          <pose>0 0 0 0 0 0</pose>
+          <visualize>false</visualize>
+          <update_rate>20</update_rate>  <!-- Controls how often (how fast) the laser data is captured -->
+          <ray>
+            <scan>
+              <horizontal>
+                <samples>360</samples>    <!-- Defines how how many readings are contained in one scan -->
+                <resolution>1</resolution> <!-- Defines the minimum angular distance between readings captured in a laser scan -->
+                <min_angle>${0}</min_angle>
+                <max_angle>${2*pi-0.01}</max_angle>
+              </horizontal>
+            </scan>
+            <range>
+              <min>0.10</min>
+              <max>18.0</max>
+              <resolution>0.01</resolution>
+            </range>
+            <noise>
+              <type>gaussian</type>
+              <mean>0.0</mean>
+              <stddev>0.01</stddev>
+            </noise>
+          </ray>
+          <plugin name="gazebo_ros_head_rplidar_controller" filename="libgazebo_ros_laser.so">
+            <topicName>/scan</topicName>
+            <frameName>sensor_laser</frameName>
+          </plugin>
+        </sensor>
+    </gazebo>
 </robot>

Commit message: with only one caster wheel

File: mnwlk3r_ros/mnwlk3r_description/urdf/mnwlk3r_base.xacro (robot description, xacro)
@@ -36,4 +36,5 @@
   </gazebo>
     <xacro:macro name="cylinder_inertia" params="mass r l">
+      <mass value="${mass}" />
       <inertia  ixx="${mass*(3*r*r+l*l)/12}" ixy = "0" ixz = "0"
                 iyy="${mass*(3*r*r+l*l)/12}" iyz = "0"
@@ -45,5 +46,6 @@
    -->
    <xacro:macro name="box_inertia" params="x y z mass">
-     <inertia ixx="${0.0833333 * mass * (y*y + z*z)}" ixy="0.0" ixz="0.0"
+    <mass value="${mass}" />
+    <inertia ixx="${0.0833333 * mass * (y*y + z*z)}" ixy="0.0" ixz="0.0"
        iyy="${0.0833333 * mass * (x*x + z*z)}" iyz="0.0"
        izz="${0.0833333 * mass * (x*x + y*y)}" />
@@ -53,8 +55,7 @@
     <pose>0 0 0.068 0 0 0</pose>
     <inertial>
-      <mass value="5"/>
-      <origin xyz="0 0 0.1" rpy="0.0 0 0"  />
+      <origin xyz="0.1 0 0.02" rpy="0.0 0 0"  />
       <!-- <inertia ixx="0.0395416666667" ixy="0" ixz="0" iyy="0.106208333333" iyz="0" izz="0.106208333333"/> -->
-      <xacro:box_inertia mass="5.2" x="0.400" y="0.280" z="0.066" />
+      <xacro:box_inertia mass="5.2" x="0.200" y="0.280" z="0.066" />
     </inertial>
     <collision name="collision_chassis">
@@ -71,10 +72,10 @@
       <material name="grey"/>
     </visual>
-    <!-- caster front left (63mm diameter) -->
-    <collision name="caster_front_left_collision">
+    <!-- caster front (63mm diameter) -->
+    <collision name="caster_front_collision">
       <!-- Z = - main wheel radius + caster wheel radius = -136/2 + 63/2 = -68 + 31.5 = -36.5mm  -->
-      <origin xyz="0.200 0.070 -0.0362"  rpy=" 0 0 0"  />
-      <geometry>
-        <sphere radius="0.0315"/>
+      <origin xyz="0.200 0.000 ${-0.136/2 + 0.050}"  rpy=" 0 0 0"  />
+      <geometry>
+        <sphere radius="0.050"/>
       </geometry>
       <surface>
@@ -90,78 +91,7 @@
     </collision>
     <visual name="caster_front_left_visual">
-      <origin xyz="0.200 0.070 -0.0362"  rpy=" 0 0 0"  />
-      <geometry>
-        <sphere radius="0.0315"/>
-      </geometry>
-    </visual>
-    <!-- caster front right  -->
-    <collision name="caster_front_right_collision">
-      <origin xyz="0.200 -0.070 -0.0362"  rpy=" 0 0 0"  />
-      <geometry>
-        <sphere radius="0.0315"/>
-      </geometry>
-      <surface>
-        <friction>
-          <ode>
-            <mu>0</mu>
-            <mu2>0</mu2>
-            <slip1>1.0</slip1>
-            <slip2>1.0</slip2>
-          </ode>
-        </friction>
-      </surface>
-    </collision>
-    <visual name="caster_front_right_visual">
-      <origin xyz="0.200 -0.070 -0.0362"  rpy=" 0 0 0"  />
-      <geometry>
-        <sphere radius="0.0315"/>
-      </geometry>
-    </visual>
-    <!-- caster back left  -->
-    <collision name="caster_back_left_collision">
-      <!-- Z = - main wheel radius + caster wheel radius = -136/2 + 63/2 = -68 + 31.5 = -36.5mm  -->
-      <origin xyz="-0.150 0.080 -0.0362"  rpy=" 0 0 0"  />
-      <geometry>
-        <sphere radius="0.0315"/>
-      </geometry>
-      <surface>
-        <friction>
-          <ode>
-            <mu>0</mu>
-            <mu2>0</mu2>
-            <slip1>1.0</slip1>
-            <slip2>1.0</slip2>
-          </ode>
-        </friction>
-      </surface>
-    </collision>
-    <visual name="caster_back_left_visual">
-      <origin xyz="-0.150 0.080 -0.0362"  rpy=" 0 0 0"  />
-      <geometry>
-        <sphere radius="0.0315"/>
-      </geometry>
-    </visual>
-    <!-- caster back right  -->
-    <collision name="caster_back_right_collision">
-      <!-- Z = - main wheel radius + caster wheel radius = -136/2 + 63/2 = -68 + 31.5 = -36.5mm  -->
-      <origin xyz="-0.150 -0.080 -0.0362"  rpy=" 0 0 0"  />
-      <geometry>
-        <sphere radius="0.0315"/>
-      </geometry>
-      <surface>
-        <friction>
-          <ode>
-            <mu>0</mu>
-            <mu2>0</mu2>
-            <slip1>1.0</slip1>
-            <slip2>1.0</slip2>
-          </ode>
-        </friction>
-      </surface>
-    </collision>
-    <visual name="caster_back_right_visual">
-      <origin xyz="-0.150 -0.080 -0.0362"  rpy=" 0 0 0"  />
-      <geometry>
-        <sphere radius="0.0315"/>
+      <origin xyz="0.200 0.000 ${-0.136/2 + 0.050}"  rpy=" 0 0 0"  />
+      <geometry>
+        <sphere radius="0.050"/>
       </geometry>
     </visual>
@@ -171,5 +101,4 @@
   <link name="link_right_wheel">
     <inertial>
-      <mass value="0.2"/>
       <origin  xyz="0 0 0" rpy="1.5707 0 0" />  <!-- only 90 deg rotation on X = pi/2 -->
       <!-- <inertia ixx="0.00052666666" ixy="0" ixz="0" iyy="0.00052666666" iyz="0" izz="0.001"/> -->
@@ -196,12 +125,20 @@
     <parent link="base_footprint"/>
     <axis  xyz="0 1 0" rpy="0 0 0" />
-    <limit effort="10000" velocity="1000"/>
+    <limit lower="0" upper="0" effort="10000" velocity="1000" />
     <joint_properties damping="1.0" friction="1.0" />
   </joint>
+  <gazebo reference="link_right_wheel">
+			<mu1 value="100000"/>
+			<mu2 value="100000"/>
+			<kp value="1000000.0" />
+			<kd value="100.0" />
+			<fdir1 value="1 0 0"/>
+			<minDepth>0.005</minDepth>
+			<gravity>true</gravity>
+	</gazebo>
   <!-- Create wheel left -->
   <!-- wheel diameter 136mm  |  width 24mm -->
   <link name="link_left_wheel">
     <inertial>
-      <mass value="0.2"/>
       <origin  xyz="0 0 0" rpy="1.5707 0 0" />  <!-- only 90 deg rotation on X = pi/2 -->
       <xacro:cylinder_inertia mass="0.150" r="${0.136/2}" l="0.024" />
@@ -227,7 +164,16 @@
     <parent link="base_footprint"/>
     <axis  xyz="0 1 0" rpy="0 0 0" />
-    <limit effort="10000" velocity="1000"/>
+    <limit lower="0" upper="0" effort="10000" velocity="1000" />
     <joint_properties damping="1.0" friction="1.0" />
   </joint>
+  <gazebo reference="link_left_wheel">
+			<mu1 value="100000"/>
+			<mu2 value="100000"/>
+			<kp value="1000000.0" />
+			<kd value="100.0" />
+			<fdir1 value="1 0 0"/>
+			<minDepth>0.005</minDepth>
+			<gravity>true</gravity>
+	</gazebo>
    <!--  *** RPLIDAR LASERSCAN ***  -->
    <!--  specs => https://www.slamtec.com/en/Lidar/A2Spec  -->
@@ -235,5 +181,4 @@
     <inertial>
       <origin xyz="0 0 0" rpy="0 0 0" />
-      <mass value="1" />
       <!-- this time we use a xacro to calculate inertia  -->
       <xacro:cylinder_inertia mass="0.190" r="0.038" l="0.041" />
@@ -267,5 +212,5 @@
          <wheelSeparation>${0.164*2}</wheelSeparation>
          <wheelDiameter>0.136</wheelDiameter>
-         <torque>0.1</torque>
+         <torque>10</torque>
          <commandTopic>cmd_vel</commandTopic>
          <odometryTopic>odom</odometryTopic>

Commit message: now mnwlk3r in gazebo feels somehow ok-ish... go figure

File: mnwlk3r_ros/mnwlk3r_description/urdf/mnwlk3r_base.xacro (robot description, xacro)
@@ -55,7 +55,6 @@
     <pose>0 0 0.068 0 0 0</pose>
     <inertial>
-      <origin xyz="0.1 0 0.02" rpy="0.0 0 0"  />
-      <!-- <inertia ixx="0.0395416666667" ixy="0" ixz="0" iyy="0.106208333333" iyz="0" izz="0.106208333333"/> -->
-      <xacro:box_inertia mass="5.2" x="0.200" y="0.280" z="0.066" />
+      <origin xyz="0.030 0 0.062" rpy="0.0 0 0"  />
+      <xacro:box_inertia mass="5.2" x="0.400" y="0.280" z="0.066" />
     </inertial>
     <collision name="collision_chassis">
@@ -96,4 +95,27 @@
       </geometry>
     </visual>
+    <!-- caster bask  -->
+    <collision name="caster_back_collision">
+      <origin xyz="-0.150 0.000 ${-0.136/2 + 0.050}"  rpy=" 0 0 0"  />
+      <geometry>
+        <sphere radius="0.050"/>
+      </geometry>
+      <surface>
+        <friction>
+          <ode>
+            <mu>0</mu>
+            <mu2>0</mu2>
+            <slip1>1.0</slip1>
+            <slip2>1.0</slip2>
+          </ode>
+        </friction>
+      </surface>
+    </collision>
+    <visual name="caster_back_left_visual">
+      <origin xyz="-0.150 0.000 ${-0.136/2 + 0.050}"  rpy=" 0 0 0"  />
+      <geometry>
+        <sphere radius="0.050"/>
+      </geometry>
+    </visual>
   </link>
   <!-- Create wheel right -->
@@ -121,5 +143,5 @@
   <!--   Joint for right wheel  -->
   <joint name="joint_right_wheel" type="continuous">
-    <origin xyz="0 -0.164 0" rpy="0 0 0"  /> <!-- X=0  |  Y = half box width + 12m spacer + half wheel width ==> x = -280/2 - 12mm -24/2 = -164mm  -->
+    <origin xyz="0 -0.164 -0.001" rpy="0 0 0"  /> <!-- X=0  |  Y = half box width + 12m spacer + half wheel width ==> x = -280/2 - 12mm -24/2 = -164mm  -->
     <child link="link_right_wheel" />
     <parent link="base_footprint"/>
@@ -160,5 +182,5 @@
   <!--   Joint for left wheel  -->
   <joint name="joint_left_wheel" type="continuous">
-    <origin xyz="0 0.164 0" rpy="0 0 0"  /> <!-- X=0  |  Y = half box width + 12m spacer + half wheel width ==> x = -280/2 - 12mm -24/2 = -164mm  -->
+    <origin xyz="0 0.164 -0.001" rpy="0 0 0"  /> <!-- X=0  |  Y = half box width + 12m spacer + half wheel width ==> x = -280/2 - 12mm -24/2 = -164mm  -->
     <child link="link_left_wheel" />
     <parent link="base_footprint"/>
